Commit message: feat: Fairino5カスタマイズ（ros2_control設定、ServoJ対応、実機launch追加）
- ros2_control.xacro/urdf.xacro: mock hardware対応、joint設定変更
- joint_limits.yaml/ros2_controllers.yaml: コントローラー設定調整
- demo.launch.py: 実機対応パラメータ追加
- demo_real.launch.py: 実機用launchファイル新規追加
- fairino_hardware_interface: ServoJ対応、初期化改善
- libfairino.so/so.2: 更新されたSDKライブラリ

File: fairino5_v6_moveit2_config/config/fairino5_v6_robot.ros2_control.xacro (robot description, xacro)
@@ -1,10 +1,17 @@
 <?xml version="1.0"?>
 <robot xmlns:xacro="http://www.ros.org/wiki/xacro">
-    <xacro:macro name="fairino5_v6_robot_ros2_control" params="name initial_positions_file">
-        <xacro:property name="initial_positions" value="${load_yaml(initial_positions_file)['initial_positions']}"/>
+    <xacro:macro name="fairino5_v6_robot_ros2_control" params="name initial_positions_file use_fake_hardware:=true robot_ip:=192.168.58.2">
+        <xacro:property name="initial_positions" value="${xacro.load_yaml(initial_positions_file)['initial_positions']}"/>
         <ros2_control name="${name}" type="system">
             <hardware>
-                <!-- By default, set up controllers for simulation. This won't work on real hardware -->
-                <plugin>mock_components/GenericSystem</plugin>
+                <xacro:if value="${use_fake_hardware}">
+                    <!-- Mock hardware for simulation/demo -->
+                    <plugin>mock_components/GenericSystem</plugin>
+                </xacro:if>
+                <xacro:unless value="${use_fake_hardware}">
+                    <!-- Real hardware interface for Fairino robot -->
+                    <plugin>fairino_hardware/FairinoHardwareInterface</plugin>
+                    <param name="robot_ip">${robot_ip}</param>
+                </xacro:unless>
             </hardware>
             <joint name="j1">

File: fairino5_v6_moveit2_config/config/fairino5_v6_robot.urdf.xacro (robot description, xacro)
@@ -2,8 +2,14 @@
 <robot xmlns:xacro="http://www.ros.org/wiki/xacro" name="fairino5_v6_robot">
     <xacro:arg name="initial_positions_file" default="initial_positions.yaml" />
+    <xacro:arg name="use_fake_hardware" default="true" />
+    <xacro:arg name="robot_ip" default="192.168.58.2" />
     <!-- Import fairino5_v6_robot urdf file -->
     <xacro:include filename="$(find fairino_description)/urdf/fairino5_v6.urdf" />
     <!-- Import control_xacro -->
     <xacro:include filename="fairino5_v6_robot.ros2_control.xacro" />
-    <xacro:fairino5_v6_robot_ros2_control name="FakeSystem" initial_positions_file="$(arg initial_positions_file)"/>
+    <xacro:fairino5_v6_robot_ros2_control
+        name="FairinoSystem"
+        initial_positions_file="$(arg initial_positions_file)"
+        use_fake_hardware="$(arg use_fake_hardware)"
+        robot_ip="$(arg robot_ip)"/>
 </robot>
